File: Crazyflie_charging_deck/Crazyflie_charging_deck.kicad_sch (KiCad schematic)
At the start: 0 parts

Commit message: Update KiCad project
Other:
- company: (none) -> University of Luxembourg - SnT
- title: (none) -> Crazyflie charging deck
Changed lines of the file:
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@@
 	(generator_version "10.0")
 	(paper "A4")
+	(title_block
+		(title "Crazyflie charging deck")
+		(date "2026-08-19")
+		(rev "A")
+		(company "University of Luxembourg - SnT")
+	)
 	(sheet_instances
 		(path "/"

Commit message: Complete Rev.A layout
Parts:
- added C1, C10, C11, C12, C2, C3, C4, C5, C6, C7, C8, C9: 100nF, crazyflie_charging_deck:C_0603_1608Metric, symbol crazyflie_charging_deck:C
- added C13, C15: 10µF, crazyflie_charging_deck:C_1206_3216Metric, symbol crazyflie_charging_deck:C
- added C14, C16: 22µF, crazyflie_charging_deck:C_1206_3216Metric, symbol crazyflie_charging_deck:C
- added D1, D10, D11, D12, D2, D3, D4, D5, D6, D7, D8, D9: WS2812B, crazyflie_charging_deck:LED_WS2812B_PLCC4_5.0x5.0mm_P3.2mm, symbol crazyflie_charging_deck:WS2812B
- added D13: MB14F_C2943867, crazyflie_charging_deck:MBF-SMD_L4.7-W3.8-P2.50-LS7.0-BL, symbol crazyflie_charging_deck:MB14F_C2943867
- added J1, J2: HX PM2.0-1X10P TP-YQ, crazyflie_charging_deck:CONN-SMD_10P-P2.00_TPYE-1_SMD-10P, symbol crazyflie_charging_deck:HXPM2.0-1X10PTP-YQ
- added L1, L2: 2.2µH, crazyflie_charging_deck:L_Sunlord_SWPA4020S, symbol crazyflie_charging_deck:L
- added R1, R4: DO NOT MOUNT, crazyflie_charging_deck:R_0603_1608Metric, symbol crazyflie_charging_deck:R
- added R2, R5: 100k, crazyflie_charging_deck:R_0603_1608Metric, symbol crazyflie_charging_deck:R
- added R3: 15k, crazyflie_charging_deck:R_0603_1608Metric, symbol crazyflie_charging_deck:R
- added R6: 11k, crazyflie_charging_deck:R_0603_1608Metric, symbol crazyflie_charging_deck:R
- added TP1, TP2: TestPoint, crazyflie_charging_deck:TestPoint_Pad_4.0x4.0mm, symbol crazyflie_charging_deck:TestPoint
- added U3: DS28E05R+T, crazyflie_charging_deck:DS28E05R+T, symbol crazyflie_charging_deck:DS28E05R+T
- added U4, U5: STBB1-APUR, crazyflie_charging_deck:STBB1-APUR, symbol crazyflie_charging_deck:STBB1-APUR
Connections:
- new net: D6.2 (DOUT), D7.4 (DIN)
- new net: D5.2 (DOUT), D6.4 (DIN)
- new net: D4.2 (DOUT), D5.4 (DIN)
- new net: D3.2 (DOUT), D4.4 (DIN)
- new net: L2.1, U5.4 (SW1)
- new net: L2.2, U5.2 (SW2)
- new net: D2.2 (DOUT), D3.4 (DIN)
- new net: R2.2, R3.1, U4.10 (FB)
- new net: D10.4 (DIN), D9.2 (DOUT)
- new net: D8.2 (DOUT), D9.4 (DIN)
- new net: R5.2, R6.1, U5.10 (FB)
- new net: D7.2 (DOUT), D8.4 (DIN)
- new net: D1.2 (DOUT), D2.4 (DIN)
- new net: D11.2 (DOUT), D12.4 (DIN)
- new net: L1.2, U4.2 (SW2)
- new net: L1.1, U4.4 (SW1)
- new net: D10.2 (DOUT), D11.4 (DIN)
- new net GND: C1.2, C10.2, C11.2, C12.2, C13.2, C14.2, C15.2, C16.2, C2.2, C3.2, C4.2, C5.2, C6.2, C7.2, C8.2, C9.2, D1.3 (VSS), D10.3 (VSS), D11.3 (VSS), D12.3 (VSS), D13.2 (-), D2.3 (VSS), D3.3 (VSS), D4.3 (VSS), D5.3 (VSS), D6.3 (VSS), D7.3 (VSS), D8.3 (VSS), D9.3 (VSS), J1.10, R3.2, R6.2, U3.3 (GND), U4.11 (EPAD), U4.3 (PGND), U4.7 (MODE/SYNC), U4.9 (GND), U5.11 (EPAD), U5.3 (PGND), U5.7 (MODE/SYNC), U5.9 (GND)
- new net IO_2: D1.4 (DIN), J1.7
- new net OW: J2.8, U3.1 (IO)
- new net VCC: C1.1, C10.1, C11.1, C12.1, C14.1, C2.1, C3.1, C4.1, C5.1, C6.1, C7.1, C8.1, C9.1, D1.1 (VDD), D10.1 (VDD), D11.1 (VDD), D12.1 (VDD), D2.1 (VDD), D3.1 (VDD), D4.1 (VDD), D5.1 (VDD), D6.1 (VDD), D7.1 (VDD), D8.1 (VDD), D9.1 (VDD), R1.1, R2.1, U4.1 (VOUT)
- new net VCOM: C13.1, J2.9, R1.2, U4.5 (VIN), U4.6 (EN), U4.8 (VINA)
- new net VPAD1: D13.3 (AC), TP1.1
- new net VPAD2: D13.4 (AC), TP2.1
- new net VPAD_RECT+: C15.1, D13.1 (+), R4.2, U5.5 (VIN), U5.6 (EN), U5.8 (VINA)
- new net VUSB: C16.1, J2.10, R4.1, R5.1, U5.1 (VOUT)
- no-connect marks 0 -> 17
Other:
- note added: "1-Wire chip"
- note added: "3.8V voltage regulator (for the LEDs)"
- note added: "5V voltage regulator (used when charging)"
- note added: "Full bridge rectifier (Schottky diodes)"
- note added: "Left header"
- note added: "Pads"
- note added: "RGB LEDs"
- note added: "Right header"
- note added: "VCC = VFB*(R2/R3 + 1) VCC = 0.5*(100/15 +1) = 3.83 V"
- note added: "VUSB = VFB*(R5/R6 + 1) VUSB = 0.5*(100/11 +1) = 5.05 V"
- note added: "When considering the Crazyflie right side up"
